File: pcb/reviung48.kicad_pcb (KiCad board)
At the start: 2 copper layers, 253.3 x 117 mm, 126 parts, among them SW1 SW_PUSH, SW10 SW_PUSH, SW11 SW_PUSH, SW12 SW_PUSH, SW13 SW_PUSH, SW14 SW_PUSH, SW15 SW_PUSH, SW16 SW_PUSH, SW17 SW_PUSH, SW18 SW_PUSH, SW19 SW_PUSH, SW2 SW_PUSH, SW20 SW_PUSH, SW21 SW_PUSH, SW22 SW_PUSH, SW23 SW_PUSH, SW24 SW_PUSH, SW25 SW_PUSH, SW26 SW_PUSH, SW27 SW_PUSH, SW28 SW_PUSH, SW29 SW_PUSH, SW3 SW_PUSH, SW30 SW_PUSH, SW31 SW_PUSH, SW32 SW_PUSH, SW33 SW_PUSH, SW34 SW_PUSH, SW35 SW_PUSH, SW36 SW_PUSH, SW37 SW_PUSH, SW38 SW_PUSH, SW39 SW_2U_PUSH, SW4 SW_PUSH, SW40 SW_2U_PUSH, SW41 SW_PUSH, SW42 SW_PUSH, SW43 SW_PUSH, SW44 SW_PUSH, SW45 SW_PUSH, SW46 SW_PUSH, SW47 SW_PUSH, SW48 SW_PUSH, SW5 SW_PUSH, SW6 SW_PUSH, SW7 SW_PUSH, SW8 SW_PUSH, SW9 SW_PUSH, U1 ProMicro

Commit message: fixed screw hole position
Parts:
- moved H1 20.3 mm to (55.0, 48.9)
- moved SW41 4.00 mm to (184.5, 129.5)
- moved ? 4.00 mm to (93.8, 48.6)
- moved D29 4.00 mm to (240.5, 82.8)
- moved SW35 4.00 mm to (242.9, 97.3)
- moved SW37 4.00 mm to (89.0, 118.4)
- moved D40 4.00 mm to (185.9, 133.7)
- moved SW27 4.00 mm to (200.8, 78.2)
- moved D6 4.00 mm to (136.4, 77.3)
- moved H4 4.00 mm to (103.3, 114.3)
- moved D13 4.00 mm to (35.3, 101.7)
- moved D2 4.00 mm to (61.4, 64.1)
- moved D7 4.00 mm to (38.8, 83.0)
- moved H5 4.00 mm to (127.1, 75.3)
- moved H9 4.00 mm to (211.6, 83.9)
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