File: pcb-top-plate/ver1.4/pcb-top-plate.kicad_pcb (KiCad board)
At the start: 2 copper layers, 253.3 x 101.2 mm, 44 parts

Commit message: finished pcb and plate
fixed edgecuts, promicro position, promicro cover and some wiring
Parts:
- added H4: MountingHole_2.2mm_M2, MountingHole:MountingHole_2.2mm_M2, F.Cu at (89.5, 49.6)
- H12, H13, H14: moved to B.Cu
- moved H12 50.1 mm to (179.1, 55.0), turned to 180 degrees
- moved H13 27.9 mm to (167.9, 57.0), turned to 180 degrees
- moved H14 26.2 mm to (141.6, 42.6), turned to 180 degrees
- moved H11 17.4 mm to (50.7, 49.9)
- moved Ref** 0.57 mm to (147.5, 83.5)
- moved Ref** 0.57 mm to (139.5, 113.7)
- moved H8 0.57 mm to (207.2, 84.9)
- moved Ref** 0.57 mm to (142.2, 89.0)
- moved H9 0.57 mm to (242.6, 66.4)
- moved H4 0.57 mm to (122.8, 76.3)
- moved Ref** 0.57 mm to (150.2, 97.2)
- moved Ref** 0.57 mm to (147.5, 100.0)
- moved Ref** 0.57 mm to (147.5, 105.5)
- moved H3 0.57 mm to (82.6, 84.9)
- moved Ref** 0.57 mm to (142.2, 105.5)
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Other:
- board size 253.3 x 101.2 mm -> 253.3 x 115.3 mm
- net class Default removed
