File: pcb-v2/reviung48.kicad_pcb (KiCad board)
At the start: 2 copper layers, 253.3 x 117 mm, 126 parts, among them SW1 SW_PUSH, SW10 SW_PUSH, SW11 SW_PUSH, SW12 SW_PUSH, SW13 SW_PUSH, SW14 SW_PUSH, SW15 SW_PUSH, SW16 SW_PUSH, SW17 SW_PUSH, SW18 SW_PUSH, SW19 SW_PUSH, SW2 SW_PUSH, SW20 SW_PUSH, SW21 SW_PUSH, SW22 SW_PUSH, SW23 SW_PUSH, SW24 SW_PUSH, SW25 SW_PUSH, SW26 SW_PUSH, SW27 SW_PUSH, SW28 SW_PUSH, SW29 SW_PUSH, SW3 SW_PUSH, SW30 SW_PUSH, SW31 SW_PUSH, SW32 SW_PUSH, SW33 SW_PUSH, SW34 SW_PUSH, SW35 SW_PUSH, SW36 SW_PUSH, SW37 SW_PUSH, SW38 SW_PUSH, SW39 SW_2U_PUSH, SW4 SW_PUSH, SW40 SW_2U_PUSH, SW41 SW_PUSH, SW42 SW_PUSH, SW43 SW_PUSH, SW44 SW_PUSH, SW45 SW_PUSH, SW46 SW_PUSH, SW47 SW_PUSH, SW48 SW_PUSH, SW5 SW_PUSH, SW6 SW_PUSH, SW7 SW_PUSH, SW8 SW_PUSH, SW9 SW_PUSH, U1 ProMicro

Commit message: finished pcb
v2 is slightly better edgecut than v1
Parts:
- moved H14 2.73 mm to (166.5, 38.1)
Routing:
- net GND: vias 25 -> 26
Other:
- outline, holes or cut-outs redrawn
Changed lines of the file:
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@@
   )
   (footprint "_reviung-kbd:HOLE_2.2mm" (layer "B.Cu")
-    (at 166.86 40.78)
+    (at 166.458029 38.079548)
     (descr "Mounting Hole 2.2mm, no annular, M2")
     (tags "mounting hole 2.2mm no annular m2")
@@
   (gr_curve (pts (xy 22.067496 110.534962) (xy 22.067496 110.534962) (xy 40.875596 113.845464) (xy 40.875596 113.845464)) (layer "Edge.Cuts") (width 0.1))
   (gr_curve (pts (xy 170.884441 147.712689) (xy 170.884441 147.712689) (xy 196.024193 140.981642) (xy 196.024193 140.981642)) (layer "Edge.Cuts") (width 0.1))
-  (gr_line (start 96.747573 30.717459) (end 180.29 40.372551) (layer "Edge.Cuts") (width 0.1))
   (gr_curve (pts (xy 96.747573 30.717459) (xy 96.747573 30.717459) (xy 35.640087 30.717333) (xy 35.640087 30.717333)) (layer "Edge.Cuts") (width 0.1))
-  (gr_arc (start 180.29 40.372551) (mid 180.817102 40.652131) (end 181.087991 41.183759) (layer "Edge.Cuts") (width 0.1))
   (gr_curve (pts (xy 242.479083 112.046748) (xy 242.479083 112.046748) (xy 250.896201 113.831984) (xy 250.896201 113.831984)) (layer "Edge.Cuts") (width 0.1))
   (gr_line (start 92.391898 133.264929) (end 74.989711 133.264929) (layer "Edge.Cuts") (width 0.1))
@@
   (gr_line (start 270.447524 110.535074) (end 251.658156 113.845174) (layer "Edge.Cuts") (width 0.1))
   (gr_curve (pts (xy 92.391898 133.264929) (xy 92.804529 133.264932) (xy 93.174789 133.518374) (xy 93.324117 133.903034)) (layer "Edge.Cuts") (width 0.1))
+  (gr_curve (pts (xy 165.688176 42.888982) (xy 114.703688 33.899044) (xy 96.747573 30.717459) (xy 96.747573 30.717459)) (layer "Edge.Cuts") (width 0.1))
   (gr_curve (pts (xy 19.633375 107.057967) (xy 19.344692 108.690427) (xy 20.434799 110.247587) (xy 22.067496 110.534962)) (layer "Edge.Cuts") (width 0.1))
   (gr_line (start 184.361515 53.98229) (end 211.965658 49.114882) (layer "Edge.Cuts") (width 0.1))
@@
   (gr_curve (pts (xy 219.381835 116.020074) (xy 219.381835 116.020074) (xy 241.712704 112.034341) (xy 241.712704 112.034341)) (layer "Edge.Cuts") (width 0.1))
   (gr_line (start 93.324117 133.903034) (end 95.837414 140.377175) (layer "Edge.Cuts") (width 0.1))
+  (gr_curve (pts (xy 179.929515 40.372551) (xy 180.473434 40.27664) (xy 180.992114 40.639838) (xy 181.087991 41.183759)) (layer "Edge.Cuts") (width 0.1))
   (gr_curve (pts (xy 73.98971 132.264928) (xy 73.989711 132.817213) (xy 74.437425 133.264929) (xy 74.989711 133.264929)) (layer "Edge.Cuts") (width 0.1))
   (gr_curve (pts (xy 41.634983 113.832707) (xy 41.634983 113.832707) (xy 50.096067 112.0484) (xy 50.096067 112.0484)) (layer "Edge.Cuts") (width 0.1))
@@
   (gr_curve (pts (xy 272.881453 107.059594) (xy 272.881453 107.059594) (xy 263.100162 51.590905) (xy 263.100162 51.590905)) (layer "Edge.Cuts") (width 0.1))
   (gr_curve (pts (xy 196.024193 140.981642) (xy 196.332458 140.89911) (xy 196.582811 140.674412) (xy 196.698064 140.376826)) (layer "Edge.Cuts") (width 0.1))
+  (gr_line (start 179.929515 40.372551) (end 165.688176 42.888982) (layer "Edge.Cuts") (width 0.1))
   (gr_line (start 151.522795 63.444358) (end 148.435329 45.934475) (layer "B.Fab") (width 0.1))
   (gr_line (start 184.021448 57.713968) (end 151.522795 63.444358) (layer "B.Fab") (width 0.1))
@@
   (via (at 182.514886 65.938635) (size 0.6) (drill 0.3) (layers "F.Cu" "B.Cu") (free) (net 51))
   (via (at 157.61006 108.042655) (size 0.6) (drill 0.3) (layers "F.Cu" "B.Cu") (free) (net 51))
+  (via (at 158.2 43.14) (size 0.6) (drill 0.3) (layers "F.Cu" "B.Cu") (free) (net 51))
   (via (at 39.604888 99.068638) (size 0.6) (drill 0.3) (layers "F.Cu" "B.Cu") (free) (net 51))
   (via (at 49.884888 84.738636) (size 0.6) (drill 0.3) (layers "F.Cu" "B.Cu") (free) (net 51))

Commit message: fixed pcb folder names
Parts:
- moved H1 20.3 mm to (55.0, 48.9)
- moved SW41 4.00 mm to (184.5, 129.5)
- moved ? 4.00 mm to (93.8, 48.6)
- moved D29 4.00 mm to (240.5, 82.8)
- moved SW35 4.00 mm to (242.9, 97.3)
- moved SW37 4.00 mm to (89.0, 118.4)
- moved D40 4.00 mm to (185.9, 133.7)
- moved SW27 4.00 mm to (200.8, 78.2)
- moved D6 4.00 mm to (136.4, 77.3)
- moved H4 4.00 mm to (103.3, 114.3)
- moved D13 4.00 mm to (35.3, 101.7)
- moved D2 4.00 mm to (61.4, 64.1)
- moved D7 4.00 mm to (38.8, 83.0)
- moved H5 4.00 mm to (127.1, 75.3)
- moved H9 4.00 mm to (211.6, 83.9)
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Routing:
- net GND: vias 26 -> 25
Other:
- outline, holes or cut-outs redrawn

Commit message: finished pcb and plate
fixed edgecuts, promicro position, promicro cover and some wiring
Parts:
- RESET1: moved to F.Cu
- moved H14 30.0 mm to (141.1, 46.8), turned to 180 degrees
- moved H12 27.0 mm to (178.6, 59.3), turned to 180 degrees
- moved H13 24.6 mm to (167.4, 61.3), turned to 180 degrees
- moved RESET1 15.1 mm to (224.4, 53.6), turned to 180 degrees
- moved D2 7.11 mm to (60.0, 50.6)
- moved SW32 7.11 mm to (181.2, 109.0)
- moved D23 7.11 mm to (232.4, 69.4)
- moved D16 7.11 mm to (88.7, 106.6)
- moved SW34 7.11 mm to (218.8, 102.4)
- moved D5 7.11 mm to (116.8, 57.1)
- moved SW15 7.11 mm to (70.1, 102.4)
- moved G*** 7.11 mm to (156.7, 145.8)
- moved D39 7.11 mm to (154.0, 142.4)
- moved D26 7.11 mm to (178.7, 94.6)
- moved D29 7.11 mm to (235.7, 88.1)
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Routing:
- net col0: track 345.6 -> 287.8 mm, vias 0 -> 4
- net col5: track 325.2 -> 372.8 mm
- net col4: track 315.5 -> 360.4 mm, vias 2 -> 1
- net reset: track 31.6 -> 55.7 mm
- net col3: track 305.0 -> 328.0 mm, vias 2 -> 3
- net col1: track 320.6 -> 300.6 mm, vias 2 -> 5
- net VCC: track 524.1 -> 517.4 mm
- net LED: track 87.5 -> 94.1 mm
- net row3: track 150.8 -> 156.3 mm
- net row4: track 176.1 -> 181.5 mm
- net row5: track 185.7 -> 191.2 mm
- net row2: track 195.6 -> 201.1 mm
- net row1: track 175.2 -> 180.5 mm
- net row0: track 162.9 -> 167.8 mm
- net row6: track 232.9 -> 236.3 mm
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Other:
- board size 253.3 x 117 mm -> 253.3 x 115.3 mm
