File: pcb-top-plate/pcb-top-plate.kicad_pcb (KiCad board)
At the start: 2 copper layers, 253.3 x 115.3 mm, 46 parts

Commit message: fixed the pcbs
Other:
- board text added: "REVIUNG48 GH"
- board text added: "REVIUNG48 GH Designed by ronzeco 2022"
- board text removed: "REVIUNG41 rev1.4 GH"
- board text removed: "REVIUNG41 rev1.4 GH Designed by gtips 2021"
Changed lines of the file:
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@@
   (gr_line (start 102.29785 71.764517) (end 102.297851 66.764518) (layer "F.Fab") (width 0.1))
   (gr_line (start 78.583973 92.505382) (end 76.170264 106.19421) (layer "F.Fab") (width 0.1))
-  (gr_text "REVIUNG41 rev1.4 GH\nDesigned by gtips 2021" (at 119.045629 123.33369 -15) (layer "B.SilkS")
+  (gr_text "REVIUNG48 GH\nDesigned by ronzeco 2022" (at 119.045629 123.33369 -15) (layer "B.SilkS")
     (effects (font (size 0.8 0.8) (thickness 0.15)) (justify left mirror))
   )
-  (gr_text "REVIUNG41 rev1.4 GH" (at 223.185629 110.87369 10) (layer "F.Mask")
+  (gr_text "REVIUNG48 GH" (at 223.185629 110.87369 10) (layer "F.Mask")
     (effects (font (size 0.85 0.85) (thickness 0.12)))
   )

Commit message: fixed pcb-plate and pic
Parts:
- moved Ref** 1.40 mm to (138.8, 92.9)
- moved H4 1.40 mm to (88.7, 50.7)
- moved Ref** 1.40 mm to (138.8, 98.4)
- moved Ref** 1.40 mm to (146.7, 112.1)
- moved Ref** 1.40 mm to (152.1, 112.1)
- moved Ref** 1.40 mm to (144.1, 98.4)
- moved Ref** 1.40 mm to (144.1, 109.4)
- moved Ref** 1.40 mm to (144.1, 87.4)
- moved H3 1.40 mm to (81.8, 86.1)
- moved H6 1.40 mm to (166.2, 77.4)
- moved Ref** 1.40 mm to (144.1, 114.9)
- moved Ref** 1.40 mm to (149.4, 98.4)
- moved H13 1.40 mm to (167.1, 58.2)
- moved Ref** 1.40 mm to (138.8, 114.9)
- moved Ref** 1.40 mm to (146.7, 101.1)
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Other:
- outline, holes or cut-outs redrawn
